Commit message: gripper update

File: tm_description/urdf/tm700.urdf.xacro (robot description, xacro)
@@ -275,17 +275,20 @@
     <property name="gripper_joint_x" value="0" />
     <property name="gripper_joint_y" value="0" />
-    <property name="gripper_joint_z" value="0.058" />
+    <property name="gripper_joint_z" value="0.15" />
     <property name="gripper_roll" value="0" />
-    <property name="gripper_pitch" value="${-pi/2}" />
-    <property name="gripper_yaw" value="${-pi/2}" />
-    <property name="finger_bias_x" value="-0.07285" />
-    <property name="finger_bias_y" value="0.005" />
-    <property name="finger_bias_z" value="0.068" />
-    <property name="finger_r_joint_x" value="${finger_bias_x+0.07285}" />
-    <property name="finger_r_joint_y" value="${finger_bias_y+0}" />
-    <property name="finger_r_joint_z" value="${finger_bias_z+0.0050143}" />
-    <property name="finger_l_joint_x" value="${finger_bias_x+0.07285}" />
-    <property name="finger_l_joint_y" value="${finger_bias_y+0}" />
-    <property name="finger_l_joint_z" value="${finger_bias_z+0.0050143}" />
+    <property name="gripper_pitch" value="${pi}" />
+    <property name="gripper_yaw" value="0" />
+    <property name="finger_roll" value="${pi}" />
+    <property name="finger_pitch" value="0" />
+    <property name="finger_yaw" value="0" />
+    <property name="finger_bias_x" value="0.0" />
+    <property name="finger_bias_y" value="0.0015" />
+    <property name="finger_bias_z" value="0.013" />
+    <property name="finger_r_joint_x" value="${finger_bias_x-0.0105}" />
+    <property name="finger_r_joint_y" value="${finger_bias_y+0.0}" />
+    <property name="finger_r_joint_z" value="${finger_bias_z+0.0}" />
+    <property name="finger_l_joint_x" value="${finger_bias_x+0.0105}" />
+    <property name="finger_l_joint_y" value="${finger_bias_y+0.0}" />
+    <property name="finger_l_joint_z" value="${finger_bias_z+0.0}" />
     <link name="${prefix}gripper_link">
         <inertial>
@@ -297,5 +300,5 @@
             <origin rpy="${gripper_roll} ${gripper_pitch} ${gripper_yaw}" xyz="0 0 0"/>
             <geometry>
-                <mesh filename="package://tm_description/meshes/gripper/gripper_link.STL"/>
+                <mesh filename="package://tm_description/meshes/toyo_gripper/Gripper.STL" scale="0.01 0.01 0.01"/>
             </geometry>
             <material name="">
@@ -306,5 +309,5 @@
             <origin rpy="${gripper_roll} ${gripper_pitch} ${gripper_yaw}" xyz="0 0 0"/>
             <geometry>
-                <mesh filename="package://tm_description/meshes/gripper/gripper_link.STL"/>
+                <mesh filename="package://tm_description/meshes/toyo_gripper/Gripper.STL" scale="0.01 0.01 0.01"/>
             </geometry>
         </collision>
@@ -324,7 +327,7 @@
         </inertial>
         <visual>
-            <origin rpy="${gripper_roll} ${gripper_pitch} ${gripper_yaw}" xyz="0 0 0"/>
-            <geometry>
-                <mesh filename="package://tm_description/meshes/gripper/finger_r.STL"/>
+            <origin rpy="${finger_roll} ${finger_pitch} ${finger_yaw}" xyz="0 0 0"/>
+            <geometry>
+                <mesh filename="package://tm_description/meshes/toyo_gripper/finger_r.STL" scale="0.01 0.01 0.01"/>
             </geometry>
             <material name="">
@@ -333,7 +336,7 @@
         </visual>
         <collision>
-            <origin rpy="${gripper_roll} ${gripper_pitch} ${gripper_yaw}" xyz="0 0 0"/>
-            <geometry>
-                <mesh filename="package://tm_description/meshes/gripper/finger_r.STL"/>
+            <origin rpy="${finger_roll} ${finger_pitch} ${finger_yaw}" xyz="0 0 0"/>
+            <geometry>
+                <mesh filename="package://tm_description/meshes/toyo_gripper/finger_r.STL" scale="0.01 0.01 0.01"/>
             </geometry>
         </collision>
@@ -354,7 +357,7 @@
         </inertial>
         <visual>
-            <origin rpy="${gripper_roll} ${gripper_pitch} ${gripper_yaw}" xyz="0 0 0"/>
-            <geometry>
-                <mesh filename="package://tm_description/meshes/gripper/finger_l.STL"/>
+            <origin rpy="${finger_roll} ${finger_pitch} ${finger_yaw}" xyz="0 0 0"/>
+            <geometry>
+                <mesh filename="package://tm_description/meshes/toyo_gripper/finger_l.STL" scale="0.01 0.01 0.01"/>
             </geometry>
             <material name="">
@@ -363,7 +366,7 @@
         </visual>
         <collision>
-            <origin rpy="${gripper_roll} ${gripper_pitch} ${gripper_yaw}" xyz="0 0 0"/>
-            <geometry>
-                <mesh filename="package://tm_description/meshes/gripper/finger_l.STL"/>
+            <origin rpy="${finger_roll} ${finger_pitch} ${finger_yaw}" xyz="0 0 0"/>
+            <geometry>
+                <mesh filename="package://tm_description/meshes/toyo_gripper/finger_l.STL" scale="0.01 0.01 0.01"/>
             </geometry>
         </collision>
@@ -422,5 +425,5 @@
             <origin rpy="0 0 0" xyz="0 0 0" />
             <geometry>
-                <mesh filename="package://tm_description/meshes/panel.STL" />
+                <mesh filename="package://tm_description/meshes/plate.STL" />
             </geometry>
             <material name="">
@@ -431,5 +434,5 @@
             <origin rpy="0 0 0" xyz="0 0 0"/>
             <geometry>
-                <mesh filename="package://tm_description/meshes/panel.STL"/>
+                <mesh filename="package://tm_description/meshes/plate.STL"/>
             </geometry>
         </collision>

Commit message: little modified

File: tm_description/urdf/tm700.urdf.xacro (robot description, xacro)
@@ -279,7 +279,7 @@
     <property name="gripper_pitch" value="${pi}" />
     <property name="gripper_yaw" value="0" />
-    <property name="finger_roll" value="${pi}" />
+    <property name="finger_roll" value="0" />
     <property name="finger_pitch" value="0" />
-    <property name="finger_yaw" value="0" />
+    <property name="finger_yaw" value="${pi}" />
     <property name="finger_bias_x" value="0.0" />
     <property name="finger_bias_y" value="0.0015" />
@@ -425,5 +425,6 @@
             <origin rpy="0 0 0" xyz="0 0 0" />
             <geometry>
-                <mesh filename="package://tm_description/meshes/plate.STL" />
+<!--                <mesh filename="package://tm_description/meshes/plate.STL" />-->
+                <box size="1.0 1.0 0.0001" />
             </geometry>
             <material name="">
@@ -434,5 +435,6 @@
             <origin rpy="0 0 0" xyz="0 0 0"/>
             <geometry>
-                <mesh filename="package://tm_description/meshes/plate.STL"/>
+<!--                <mesh filename="package://tm_description/meshes/plate.STL"/>-->
+                <box size="1.0 1.0 0.0001" />
             </geometry>
         </collision>
